File: Esquemático_UNCargador/Potencia.kicad_sch (KiCad schematic)
At the start: 11 parts

Commit message: Actualizacion 23-03-23
Parts:
- gave numbers to parts that had none: 11
Changed lines of the file:
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@@
     (effects (font (size 1.27 1.27)) (justify left bottom))
   )
-  (label "12V" (at 154.94 67.31 90)
+  (label "12V" (at 154.94 67.31 0)
     (effects (font (size 1.27 1.27)) (justify left bottom))
   )
   (symbol (lib_id "LED:IR26-21C_L110_TR8") (at 240.03 120.65 90) (unit 1)
     (in_bom yes) (on_board yes) (fields_autoplaced)
-    (property "Reference" "D?" (id 0) (at 243.84 120.9674 90)
+    (property "Reference" "D4" (id 0) (at 243.84 120.9674 90)
       (effects (font (size 1.27 1.27)) (justify right))
     )
@@
   (symbol (lib_id "Regulator_Linear:AMS1117-3.3") (at 177.8 113.03 0) (unit 1)
     (in_bom yes) (on_board yes) (fields_autoplaced)
-    (property "Reference" "U?" (id 0) (at 177.8 105.41 0))
+    (property "Reference" "U2" (id 0) (at 177.8 105.41 0))
     (property "Value" "AMS1117-3.3" (id 1) (at 177.8 107.95 0))
     (property "Footprint" "Package_TO_SOT_SMD:SOT-223-3_TabPin2" (id 2) (at 177.8 107.95 0)
@@
   (symbol (lib_id "power:GND") (at 177.8 129.54 0) (unit 1)
     (in_bom yes) (on_board yes) (fields_autoplaced)
-    (property "Reference" "#PWR?" (id 0) (at 177.8 135.89 0)
+    (property "Reference" "#PWR0106" (id 0) (at 177.8 135.89 0)
       (effects (font (size 1.27 1.27)) hide)
     )
@@
   (symbol (lib_id "Regulator_Linear:AMS1117-5.0") (at 177.8 73.66 0) (unit 1)
     (in_bom yes) (on_board yes) (fields_autoplaced)
-    (property "Reference" "U?" (id 0) (at 177.8 66.04 0))
+    (property "Reference" "U1" (id 0) (at 177.8 66.04 0))
     (property "Value" "AMS1117-5.0" (id 1) (at 177.8 68.58 0))
     (property "Footprint" "Package_TO_SOT_SMD:SOT-223-3_TabPin2" (id 2) (at 177.8 68.58 0)
@@
   (symbol (lib_id "Device:C_Polarized_US") (at 201.93 119.38 0) (unit 1)
     (in_bom yes) (on_board yes)
-    (property "Reference" "C?" (id 0) (at 207.01 119.38 0)
+    (property "Reference" "C5" (id 0) (at 207.01 119.38 0)
       (effects (font (size 1.27 1.27)) (justify left))
     )
@@
   (symbol (lib_id "Diode:1N4007") (at 104.14 73.66 180) (unit 1)
     (in_bom yes) (on_board yes) (fields_autoplaced)
-    (property "Reference" "D?" (id 0) (at 104.14 67.31 0))
+    (property "Reference" "D3" (id 0) (at 104.14 67.31 0))
     (property "Value" "1N4007" (id 1) (at 104.14 69.85 0))
     (property "Footprint" "Diode_SMD:D_SMA_Handsoldering" (id 2) (at 104.14 69.215 0)
@@
   (symbol (lib_id "power:GND") (at 73.66 92.71 0) (unit 1)
     (in_bom yes) (on_board yes) (fields_autoplaced)
-    (property "Reference" "#PWR?" (id 0) (at 73.66 99.06 0)
+    (property "Reference" "#PWR0101" (id 0) (at 73.66 99.06 0)
       (effects (font (size 1.27 1.27)) hide)
     )
@@
   (symbol (lib_id "Device:C_Polarized_US") (at 123.19 82.55 0) (unit 1)
     (in_bom yes) (on_board yes) (fields_autoplaced)
-    (property "Reference" "C?" (id 0) (at 127 80.6449 0)
+    (property "Reference" "C1" (id 0) (at 127 80.6449 0)
       (effects (font (size 1.27 1.27)) (justify left))
     )
@@
   (symbol (lib_id "power:GND") (at 240.03 125.73 0) (unit 1)
     (in_bom yes) (on_board yes) (fields_autoplaced)
-    (property "Reference" "#PWR?" (id 0) (at 240.03 132.08 0)
+    (property "Reference" "#PWR0109" (id 0) (at 240.03 132.08 0)
       (effects (font (size 1.27 1.27)) hide)
     )
@@
   (symbol (lib_id "power:GND") (at 123.19 92.71 0) (unit 1)
     (in_bom yes) (on_board yes) (fields_autoplaced)
-    (property "Reference" "#PWR?" (id 0) (at 123.19 99.06 0)
+    (property "Reference" "#PWR0102" (id 0) (at 123.19 99.06 0)
       (effects (font (size 1.27 1.27)) hide)
     )
@@
   (symbol (lib_id "power:+3.3V") (at 201.93 107.95 0) (unit 1)
     (in_bom yes) (on_board yes) (fields_autoplaced)
-    (property "Reference" "#PWR?" (id 0) (at 201.93 111.76 0)
+    (property "Reference" "#PWR0104" (id 0) (at 201.93 111.76 0)
       (effects (font (size 1.27 1.27)) hide)
     )
@@
   (symbol (lib_id "power:GND") (at 177.8 90.17 0) (unit 1)
     (in_bom yes) (on_board yes) (fields_autoplaced)
-    (property "Reference" "#PWR?" (id 0) (at 177.8 96.52 0)
+    (property "Reference" "#PWR0105" (id 0) (at 177.8 96.52 0)
       (effects (font (size 1.27 1.27)) hide)
     )
@@
   (symbol (lib_id "power:+3.3V") (at 240.03 106.68 0) (unit 1)
     (in_bom yes) (on_board yes) (fields_autoplaced)
-    (property "Reference" "#PWR?" (id 0) (at 240.03 110.49 0)
+    (property "Reference" "#PWR0108" (id 0) (at 240.03 110.49 0)
       (effects (font (size 1.27 1.27)) hide)
     )
@@
   (symbol (lib_id "Device:C_Polarized_US") (at 158.75 119.38 0) (unit 1)
     (in_bom yes) (on_board yes)
-    (property "Reference" "C?" (id 0) (at 151.13 116.84 0)
+    (property "Reference" "C3" (id 0) (at 151.13 116.84 0)
       (effects (font (size 1.27 1.27)) (justify left))
     )
@@
   (symbol (lib_id "Jumper:Jumper_3_Open") (at 80.01 68.58 0) (unit 1)
     (in_bom yes) (on_board yes) (fields_autoplaced)
-    (property "Reference" "JP?" (id 0) (at 80.01 62.23 0))
+    (property "Reference" "JP1" (id 0) (at 80.01 62.23 0))
     (property "Value" "Jumper_3_Open" (id 1) (at 80.01 64.77 0))
     (property "Footprint" "Connector_PinHeader_2.54mm:PinHeader_1x03_P2.54mm_Vertical" (id 2) (at 80.01 68.58 0)
@@
   (symbol (lib_id "power:+12V") (at 123.19 67.31 0) (unit 1)
     (in_bom yes) (on_board yes) (fields_autoplaced)
-    (property "Reference" "#PWR?" (id 0) (at 123.19 71.12 0)
+    (property "Reference" "#PWR0103" (id 0) (at 123.19 71.12 0)
       (effects (font (size 1.27 1.27)) hide)
     )
@@
   (symbol (lib_id "Device:C_Polarized_US") (at 154.94 80.01 0) (unit 1)
     (in_bom yes) (on_board yes)
-    (property "Reference" "C?" (id 0) (at 147.32 77.47 0)
+    (property "Reference" "C2" (id 0) (at 147.32 77.47 0)
       (effects (font (size 1.27 1.27)) (justify left))
     )
@@
   (symbol (lib_id "Device:C_Polarized_US") (at 201.93 80.01 0) (unit 1)
     (in_bom yes) (on_board yes)
-    (property "Reference" "C?" (id 0) (at 207.01 80.01 0)
+    (property "Reference" "C4" (id 0) (at 207.01 80.01 0)
       (effects (font (size 1.27 1.27)) (justify left))
     )
@@
   (symbol (lib_id "power:+5V") (at 201.93 68.58 0) (unit 1)
     (in_bom yes) (on_board yes) (fields_autoplaced)
-    (property "Reference" "#PWR?" (id 0) (at 201.93 72.39 0)
+    (property "Reference" "#PWR0107" (id 0) (at 201.93 72.39 0)
       (effects (font (size 1.27 1.27)) hide)
     )
@@
   (symbol (lib_id "Device:R") (at 240.03 111.76 0) (unit 1)
     (in_bom yes) (on_board yes) (fields_autoplaced)
-    (property "Reference" "R?" (id 0) (at 242.57 110.4899 0)
-      (effects (font (size 1.27 1.27)) (justify left))
-    )
+    (property "Reference" "R1" (id 0) (at 242.57 110.4899 0)
+      (effects (font (size 1.27 1.27)) (justify left))
+    )
