File: Esquemático_UNCargador/untitled.kicad_sch (KiCad schematic)
At the start: 0 parts

Commit message: Actualización DC-DC
Parts:
- added C2, C?: 220u, symbol Device:C
- added C?: 22uF, Capacitor_SMD:C_0805_2012Metric_Pad1.18x1.45mm_HandSolder, symbol Device:C_Polarized_US
- added Cin, Cin?: 680u, symbol Device:C
- added D1, D?: 1N5822, Diode_THT:D_DO-201AD_P15.24mm_Horizontal, symbol Diode:1N5822
- added D?: 1N4007, Diode_SMD:D_SMA_Handsoldering, symbol Diode:1N4007
- added JP?: Jumper_3_Open, Connector_PinHeader_2.54mm:PinHeader_1x03_P2.54mm_Vertical, symbol Jumper:Jumper_3_Open
- added L1, L?: 33u, symbol Device:L
- added U?: LM2596S-3.3, Package_TO_SOT_SMD:TO-263-5_TabPin3, symbol Regulator_Switching:LM2596S-3.3
- added U?: LM2596S-5, Package_TO_SOT_SMD:TO-263-5_TabPin3, symbol Regulator_Switching:LM2596S-5
Connections:
- new net: D?.1 (K), L?.1, U?.2 (OUT)
- new net: D1.1 (K), L1.1, U?.2 (OUT)
- new net: D?.2 (A), JP?.3 (B)
- new net +12V: C?.1, Cin.1, Cin?.1, D?.1 (K), U?.1 (VIN), U?.1 (VIN)
- new net +3.3V: C2.1, L1.2, U?.4 (FB)
- new net +5V: C?.1, L?.2, U?.4 (FB)
- new net GND: C2.2, C?.2, C?.2, Cin.2, Cin?.2, D1.2 (A), D?.2 (A), U?.3 (GND), U?.3 (GND), U?.5 (~{ON}/OFF), U?.5 (~{ON}/OFF)
Other:
- note added: "Contiene un filtro de condensador para eliminar cualquier tipo de rizado"
- note added: "Entrada de alimentación luego de la etapa de conversión AC-DC"

Commit message: Notacion
Parts:
- gave numbers to parts that had none: 8
- renumbered C2 to COut1, Cin to Cin1
Changed lines of the file:
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@@
   (symbol (lib_id "Device:L") (at 223.52 109.22 90) (unit 1)
     (in_bom yes) (on_board yes)
-    (property "Reference" "L?" (id 0) (at 223.52 106.68 90))
+    (property "Reference" "L2" (id 0) (at 223.52 106.68 90))
     (property "Value" "33u" (id 1) (at 223.52 111.76 90))
     (property "Footprint" "" (id 2) (at 223.52 109.22 0)
@@
   (symbol (lib_id "Device:C") (at 165.1 113.03 0) (unit 1)
     (in_bom yes) (on_board yes) (fields_autoplaced)
-    (property "Reference" "Cin?" (id 0) (at 168.91 111.7599 0)
+    (property "Reference" "CIn2" (id 0) (at 168.91 111.7599 0)
       (effects (font (size 1.27 1.27)) (justify left))
     )
@@
   (symbol (lib_id "Regulator_Switching:LM2596S-3.3") (at 194.31 54.61 0) (unit 1)
     (in_bom yes) (on_board yes) (fields_autoplaced)
-    (property "Reference" "U?" (id 0) (at 194.31 44.45 0))
+    (property "Reference" "U3.3" (id 0) (at 194.31 44.45 0))
     (property "Value" "LM2596S-3.3" (id 1) (at 194.31 46.99 0))
     (property "Footprint" "Package_TO_SOT_SMD:TO-263-5_TabPin3" (id 2) (at 195.58 60.96 0)
@@
   (symbol (lib_id "Device:C_Polarized_US") (at 120.65 91.44 0) (unit 1)
     (in_bom yes) (on_board yes) (fields_autoplaced)
-    (property "Reference" "C?" (id 0) (at 124.46 89.5349 0)
+    (property "Reference" "CIn0" (id 0) (at 124.46 89.5349 0)
       (effects (font (size 1.27 1.27)) (justify left))
     )
@@
   (symbol (lib_id "Device:C") (at 233.68 115.57 0) (unit 1)
     (in_bom yes) (on_board yes) (fields_autoplaced)
-    (property "Reference" "C?" (id 0) (at 237.49 114.2999 0)
+    (property "Reference" "COut2" (id 0) (at 237.49 114.2999 0)
       (effects (font (size 1.27 1.27)) (justify left))
     )
@@
   (symbol (lib_id "Device:C") (at 165.1 60.96 0) (unit 1)
     (in_bom yes) (on_board yes) (fields_autoplaced)
-    (property "Reference" "Cin" (id 0) (at 168.91 59.6899 0)
+    (property "Reference" "Cin1" (id 0) (at 168.91 59.6899 0)
       (effects (font (size 1.27 1.27)) (justify left))
     )
@@
   (symbol (lib_id "Device:C") (at 233.68 63.5 0) (unit 1)
     (in_bom yes) (on_board yes) (fields_autoplaced)
-    (property "Reference" "C2" (id 0) (at 237.49 62.2299 0)
+    (property "Reference" "COut1" (id 0) (at 237.49 62.2299 0)
       (effects (font (size 1.27 1.27)) (justify left))
     )
@@
   (symbol (lib_id "Regulator_Switching:LM2596S-5") (at 194.31 106.68 0) (unit 1)
     (in_bom yes) (on_board yes) (fields_autoplaced)
-    (property "Reference" "U?" (id 0) (at 194.31 96.52 0))
+    (property "Reference" "U5" (id 0) (at 194.31 96.52 0))
     (property "Value" "LM2596S-5" (id 1) (at 194.31 99.06 0))
     (property "Footprint" "Package_TO_SOT_SMD:TO-263-5_TabPin3" (id 2) (at 195.58 113.03 0)
@@
   (symbol (lib_id "Diode:1N5822") (at 212.09 115.57 270) (unit 1)
     (in_bom yes) (on_board yes) (fields_autoplaced)
-    (property "Reference" "D?" (id 0) (at 214.63 113.9824 90)
+    (property "Reference" "D2" (id 0) (at 214.63 113.9824 90)
       (effects (font (size 1.27 1.27)) (justify left))
     )
@@
   (symbol (lib_id "Diode:1N4007") (at 101.6 82.55 180) (unit 1)
     (in_bom yes) (on_board yes) (fields_autoplaced)
-    (property "Reference" "D?" (id 0) (at 101.6 76.2 0))
+    (property "Reference" "DIn" (id 0) (at 101.6 76.2 0))
     (property "Value" "1N4007" (id 1) (at 101.6 78.74 0))
     (property "Footprint" "Diode_SMD:D_SMA_Handsoldering" (id 2) (at 101.6 78.105 0)

Commit message: Actualizacion 23-03-23
Parts:
- added PS7: HLK-PM01, Convertidor_AC-DC:AC-DC_Converter, symbol Converter_ACDC:HLK-PM01
- CIn2, COut1, COut2: footprint (none) -> Capacitor_SMD:C_0201_0603Metric
- Cin1: footprint (none) -> Capacitor_SMD:C_0805_2012Metric_Pad1.18x1.45mm_HandSolder
- L1, L2: footprint (none) -> Inductor_SMD:L_Coilcraft_XxL4040
- gave numbers to parts that had none: 1
- renumbered DIn to DIn1
Other:
- moved on the sheet: CIn0, CIn2, COut1, COut2, Cin1, D1, D2, DIn1, JP2, L1, L2, U3.3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
